Commit message: feat: add aba, forward dynamics

File: tests/data/oracle_mixed.urdf (robot description, URDF)
Before this commit: robot oracle_mixed, 5 links, 4 joints
Links:
- link base: mass None -> 1.2

File: tests/data/test_arm.urdf (robot description, URDF)
Before this commit: robot test_arm, 5 links, 4 joints
Links:
- link test_base_link: mass None -> 1

File: tests/data/test_arm_40.urdf (robot description, URDF)
Before this commit: robot test_arm_40, 41 links, 40 joints
Links:
- link test_base_link: mass None -> 0.5

File: tests/data/test_tree_7.urdf (robot description, URDF)
Before this commit: robot test_tree_7, 8 links, 7 joints
Links:
- link base: mass None -> 0.8
